File: hardware/circuit.kicad_sch (KiCad schematic)
At the start: 10 parts, among them J4 AM32 dual ESC, U1 Seeed XIAO RP2350, U7 BetaFPV ELRS Lite

Commit message: feat: swap to the 74HC595 for cs expansion
Connections:
- net EXP_CS_N: no longer U1.4 (D3/A3/GPIO43)
- net LED_OE_N: no longer U1.3 (D2/A2/GPIO42)
- new net SEL_LAT: U1.4 (D3/A3/GPIO43)
- new net SEL_OE_N: U1.3 (D2/A2/GPIO42)
Other:
- sheet IMU Array ports: added LED_OE_N, SEL_LAT, SEL_OE_N; removed none
- moved on the sheet: U7

Commit message: feat: first bit of routing and double leds + fixes
Parts:
- J4: footprint Connector_Wire:SolderWire-0.25sqmm_1x04_P4.2mm_D0.65mm_OD1.7mm_Relief -> Connector_Wire:SolderWire-0.25sqmm_1x04_P4.2mm_D0.65mm_OD1.7mm
Other:
- sheet Status Leds ports: added HEAD_LED; removed none
Changed lines of the file:
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@@
+	(wire
+		(pts
+			(xy 52.07 95.25) (xy 53.34 95.25)
+		)
+		(stroke
+			(width 0)
+			(type default)
+		)
+	)
 	(wire
 		(pts
@@
 	(label "EXP_CS_N"
 		(at 53.34 60.96 0)
+		(effects
+			(font
+				(size 1.27 1.27)
+			)
+			(justify left bottom)
+		)
+	)
+	(label "HEAD_LED"
+		(at 53.34 95.25 0)
 		(effects
 			(font
@@
 			)
 		)
-		(property "Footprint" "Connector_Wire:SolderWire-0.25sqmm_1x04_P4.2mm_D0.65mm_OD1.7mm_Relief"
+		(property "Footprint" "Connector_Wire:SolderWire-0.25sqmm_1x04_P4.2mm_D0.65mm_OD1.7mm"
 			(at 149.86 86.36 0)
 			(hide yes)
@@
 			(effects
 				(font
+					(size 1.27 1.27)
+				)
+				(justify right)
+			)
+		)
+		(pin "HEAD_LED" input
+			(at 52.07 95.25 0)
+			(effects
+				(font

Commit message: feat: add bom placement
Parts:
- J4, TP13, TP14, TP15, U1, U7: now left out of the parts list
- R12, R13: LCSC Part NONE -> C3008986
Changed lines of the file:
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@@
 		(body_style 1)
 		(exclude_from_sim no)
-		(in_bom yes)
-		(on_board yes)
-		(in_pos_files yes)
+		(in_bom no)
+		(on_board yes)
+		(in_pos_files no)
 		(dnp no)
 		(fields_autoplaced yes)
@@
 			)
 		)
-		(property "LCSC Part" "NONE"
+		(property "LCSC Part" "C3008986"
 			(at -31.75 -104.14 0)
 			(hide yes)
@@
 		(body_style 1)
 		(exclude_from_sim no)
-		(in_bom yes)
-		(on_board yes)
-		(in_pos_files yes)
+		(in_bom no)
+		(on_board yes)
+		(in_pos_files no)
 		(dnp no)
 		(fields_autoplaced yes)
@@
 		(body_style 1)
 		(exclude_from_sim no)
-		(in_bom yes)
-		(on_board yes)
-		(in_pos_files yes)
+		(in_bom no)
+		(on_board yes)
+		(in_pos_files no)
 		(dnp no)
 		(property "Reference" "U1"
@@
 		(body_style 1)
 		(exclude_from_sim no)
-		(in_bom yes)
-		(on_board yes)
-		(in_pos_files yes)
+		(in_bom no)
+		(on_board yes)
+		(in_pos_files no)
 		(dnp no)
 		(fields_autoplaced yes)
@@
 			)
 		)
-		(property "LCSC Part" "NONE"
+		(property "LCSC Part" "C3008986"
 			(at -31.75 -106.68 0)
 			(hide yes)
@@
 		(body_style 1)
 		(exclude_from_sim no)
-		(in_bom yes)
-		(on_board yes)
-		(in_pos_files yes)
+		(in_bom no)
+		(on_board yes)
+		(in_pos_files no)
 		(dnp no)
 		(fields_autoplaced yes)
@@
 		(body_style 1)
 		(exclude_from_sim no)
-		(in_bom yes)
-		(on_board yes)
-		(in_pos_files yes)
+		(in_bom no)
+		(on_board yes)
+		(in_pos_files no)
 		(dnp no)
 		(fields_autoplaced yes)
