File: hardware/schm/power.kicad_sch (KiCad schematic)
At the start: 18 parts, among them J1 VBUS input fly-leads, U2 AP63205WU-7

Commit message: bug: fix lcsc inductor part number
Parts:
- L1: LCSC Part C2041623 -> C2045367
Changed lines of the file:
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@@
 			)
 		)
-		(property "LCSC Part" "C2041623"
+		(property "LCSC Part" "C2045367"
 			(at 62.23 5.08 0)
 			(hide yes)
