File: hardware/schm/power.kicad_sch (KiCad schematic)
At the start: 18 parts, among them J1 VBUS input fly-leads, U2 AP63205WU-7

Commit message: feat: update pcb to use new components
Parts:
- added C18: 47pf, Capacitor_SMD:C_0402_1005Metric, symbol Device:C_Small
- added C19, C20: 22uf, Capacitor_SMD:C_0805_2012Metric, symbol Device:C_Small
- added R27: 158kΩ, Resistor_SMD:R_0402_1005Metric, symbol Device:R_Small
- added R28: 30.1kΩ, Resistor_SMD:R_0402_1005Metric, symbol Device:R_Small
- L1: value 4.7uH -> 5.6uH; footprint Inductor_SMD:L_Wuerth_MAPI-4020 -> Inductor_SMD:L_Bourns_SRP6060FA; LCSC Part C2045367 -> Bourns SRP6060FA-5R6M
- U2: value AP63205WU-7 -> AP63300WU-7; LCSC Part C2071056 -> AP63300WU-7
Connections:
- net 5V: now also C18.2, R27.1; no longer U2.1 (FB)
- net GND: now also C19.2, C20.2, R28.2
- net VBUS: now also C19.1, C20.1
- new net BUCK_FB: C18.1, R27.2, R28.1, U2.1 (FB)
Other:
- moved on the sheet: C1, C2
